File: hardware/front_panel/FrontPanel.kicad_sch (KiCad schematic)
At the start: 95 parts, among them J1 FTSH-105-01-L-DV-K, J3 FFC2B35-10-T, SW2 TACT, SW6 ENCODER 24IMP, U1 SSD1302, U3 VSOP38338, U4 AMS1117-3.3, U5 SSD1302Z_HALF, U7 SSD1302Z_HALF, U8 STM32F103RCTx, Y1 32.768 kHz

Commit message: Prepare PCB for production
Parts:
- BT1: Manufacturer_Part_Number (none) -> BAT-HLD-012-SMT
- C1, C11, C13, C15, C2, C20, C23, C24, C25, C27, C3, C32, C34, C36, C39, C4, C40, C43, C44, C45, C46, C47, C48, C51, C8: Manufacturer_Part_Number (none) -> 0805B104K500CT
- C10, C9: Manufacturer_Part_Number (none) -> 293D106X9010A2TE3
- C12, C17, C18, C19, C21, C28, C30, C37, C49: Manufacturer_Part_Number (none) -> CL10B105KA8NNNC
- C16, C31: Manufacturer_Part_Number (none) -> CL10A475KO8NNNC
- C22: Manufacturer_Part_Number (none) -> CL10B224KO8NNNC
- C38, C50: Manufacturer_Part_Number (none) -> CL10C220JB8NNNC
- J3: Manufacturer_Part_Number (none) -> FFC2B35-10-T
- R1: Manufacturer_Part_Number (none) -> RC0603FR-07100RL
- R10, R15, R16, R2, R20, R21, R3, R4, R5, R8: Manufacturer_Part_Number (none) -> CRCW06031M00FKEA
- R11, R12, R17, R18, R19, R9: Manufacturer_Part_Number (none) -> RC0603FR-0710KL
- R13, SW2, U1, U8: now left out of the parts list
- R14: Manufacturer_Part_Number (none) -> WR06X3900FTL
- R6, R7: Manufacturer_Part_Number (none) -> RC0603FR-0749R9L
- U4: Manufacturer_Part_Number (none) -> LD1117S33TR
Other:
- note removed: "czy ffc nie sa odwrotnie"
