File: hardware/mainboard/DigitalAmplifier.kicad_pcb (KiCad board)
At the start: 6 copper layers, 178.1 x 97.2 mm, 320 parts, among them J1 FTSH-105-01-L-DV-K, J10 FFC2B35-10-T, J12 Conn_01x02, J2 Conn_01x02, J3 Conn_01x02, J4 Conn_01x02, J5 USB4215-03-A_REVA, J6 Conn_01x02, J7 43045-0414, J9 Conn_01x02, Q1 2N7002, Q2 STL130N4LF8, U1 ORJ-3__FCR6842032R_, U10 AD8694, U12 OPA2365AID, U15 STM32F446RETx, U16 SPX5205M5-L_TR, U17 OPA2188AIDR, U18 TAC5242IRGER, U19 L7987, U2 ESP32-WROOM-32UE, U3 L5973D, U4 24LC512, U5 AD8694, U6 SPX5205M5-L_TR, U7 SPX5205M5-L_TR, U9 SPX5205M5-L_TR, Y1 ASDMB-24.576MHZ-LY-T, Y2 3225-25M-SR

Commit message: Prepare PCB for production
Parts:
- removed J12, J6: Conn_01x02, digital_amp:RF219AT0050G
- J3, J4: value Conn_01x02 -> 3P HEADER; footprint digital_amp:RF219AT0050G -> Connector_JST:JST_PH_B3B-PH-K_1x03_P2.00mm_Vertical
- moved D5 5.40 mm to (94.9, 70.2), turned to 180 degrees
- moved J4 5.15 mm to (112.6, 66.7)
- moved D10 3.39 mm to (116.8, 70.3)
- moved J3 3.21 mm to (90.7, 66.7)
- moved D11 2.59 mm to (112.4, 70.3)
- moved R116 1.87 mm to (81.5, 70.7), turned to 180 degrees
- moved C11 1.87 mm to (81.5, 69.2), turned to 180 degrees
- moved C12 0.94 mm to (88.0, 123.8)
- moved R117 0.94 mm to (86.5, 123.8)
- moved D4 0.87 mm to (90.9, 70.2)
- moved U1 0.60 mm to (139.3, 69.7)
- moved C111 0.59 mm to (143.5, 75.8)
- moved FB3 0.59 mm to (146.5, 74.3)
- moved C113 0.59 mm to (143.6, 74.3)
- moved C112 0.57 mm to (138.5, 74.3)
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Connections:
- J4 pad 1: /Codec & Frontend/RCA_IN_R -> /Codec & Frontend/RCA_IN_L
Routing:
- net /Codec & Frontend/PREOUT_L: track 10.9 -> 16.0 mm
- net /Codec & Frontend/RCA_IN_R: track 12.1 -> 15.0 mm
- net /Codec & Frontend/RCA_IN_L: track 8.73 -> 9.73 mm
- net GND: track 102.3 -> 102.2 mm, vias 869 -> 851
Other:
- outline, holes or cut-outs redrawn
- board text added: "DIGITAL AMPLIFIER MAINBOARD PCB - 1 OF 3 DESIGNED BY SEWERYN SKRZYPIK 2026-05-30"
- board text removed: "DIGITAL AMPLIFIER MAINBOARD PCB - 1 OF 3 DESIGNED BY SEWERYN SKRZYPIK 2026-05-22"
