File: hardware/mainboard/mcu.kicad_sch (KiCad schematic)
At the start: 42 parts, among them J1 FTSH-105-01-L-DV-K, Q1 2N7002, U15 STM32F446RETx, U2 ESP32-WROOM-32UE, U4 24LC512, Y2 3225-25M-SR

Commit message: Add power supply and front panel PCBs
Parts:
- removed R1, R102, R31, R35, R36, R6: 0R, Resistor_SMD:R_0603_1608Metric, symbol Device:R_Small
Connections:
- net ADC_SDATA: now also U15.9 (PC1)
- net DAC_SDATA: now also U15.23 (PA7)
- net IIS3_BCLK: now also U15.51 (PC10)
- net IIS3_LRCLK: now also U15.50 (PA15)
- net IIS3_SDATA: now also U15.26 (PB0)
- net IIS_CLK: now also U15.40 (PC9)

Commit message: Prepare PCB for production
Parts:
- C107, C108: Manufacturer_Part_Number (none) -> CC0603JRNPO9BN330
- C109, C13, C15, C16, C17, C18, C35, C37: Manufacturer_Part_Number (none) -> 0603B104K500CT
- C110: Manufacturer_Part_Number (none) -> CL10A475KP8NNNC
- C14, C36, C38: Manufacturer_Part_Number (none) -> GRM188R61E106KA73J
- JP1, JP2: Manufacturer_Part_Number (none) -> DS1031-01-1*2P8BV3-1
- Q1: Manufacturer_Part_Number (none) -> 2N7002-G
- R101, R32, R34, R39: Manufacturer_Part_Number (none) -> RC0603JR-070RL
- R2, R21, R37, R5, R51, R52, R54, R56: Manufacturer_Part_Number (none) -> RC0603JR-0710KL
- R53: now left out of the parts list
- R55: Manufacturer_Part_Number (none) -> RC0603FR-07470KL
- U15: Manufacturer_Part_Number (none) -> STM32F446RETx; now left out of the parts list
- U2: Manufacturer_Part_Number (none) -> ESP32-WROOM-32UE
- U4: Manufacturer_Part_Number (none) -> 24LC512-I/SN
- Y2: Manufacturer_Part_Number (none) -> 3225-25M-SR
